File: hacker-card.kicad_sch (KiCad schematic)
At the start: 8 parts, among them U1 NT3H2111W0FHKH

Commit message: finishing up pcb journal entry
Parts:
- R1, R2, R3: value 470 -> 150; LSC C23182 -> C22808
Connections:
- net ANT_A: now reaches U1.1 (LA)
- net ANT_A: now also U1.8 (LB)
Changed lines of the file:
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@@
+	)
+	(junction
+		(at 53.34 62.23)
+		(diameter 0)
+		(color 0 0 0 0)
+	)
+	(junction
+		(at 83.82 62.23)
+		(diameter 0)
+		(color 0 0 0 0)
 	)
 	(junction
@@
 	(wire
 		(pts
-			(xy 80.01 59.69) (xy 87.63 59.69)
+			(xy 80.01 59.69) (xy 83.82 59.69)
+		)
+		(stroke
+			(width 0)
+			(type default)
+		)
+	)
+	(wire
+		(pts
+			(xy 53.34 62.23) (xy 59.69 62.23)
 		)
 		(stroke
@@
 	(wire
 		(pts
-			(xy 55.88 59.69) (xy 59.69 59.69)
+			(xy 53.34 59.69) (xy 59.69 59.69)
 		)
 		(stroke
@@
 	(wire
 		(pts
-			(xy 80.01 62.23) (xy 87.63 62.23)
+			(xy 80.01 62.23) (xy 83.82 62.23)
 		)
 		(stroke
@@
 	(wire
 		(pts
-			(xy 57.15 62.23) (xy 59.69 62.23)
-		)
-		(stroke
-			(width 0)
-			(type default)
+			(xy 46.99 62.23) (xy 53.34 62.23)
+		)
+		(stroke
+			(width 0)
+			(type default)
+		)
+	)
+	(wire
+		(pts
+			(xy 83.82 62.23) (xy 87.63 62.23)
+		)
+		(stroke
+			(width 0)
+			(type default)
+		)
+	)
+	(label "ANT_A"
+		(at 83.82 59.69 0)
+		(effects
+			(font
+				(size 1.27 1.27)
+			)
+			(justify left bottom)
+		)
+	)
+	(label "ANT_A"
+		(at 53.34 59.69 0)
+		(effects
+			(font
+				(size 1.27 1.27)
+			)
+			(justify left bottom)
 		)
 	)
 	(symbol
 		(lib_id "power:GND")
-		(at 57.15 62.23 270)
+		(at 46.99 62.23 270)
 		(unit 1)
 		(body_style 1)
@@
 		(fields_autoplaced yes)
 		(property "Reference" "#PWR01"
-			(at 50.8 62.23 0)
+			(at 40.64 62.23 0)
 			(hide yes)
 			(show_name no)
@@
 		)
 		(property "Value" "GND"
-			(at 53.34 62.2299 90)
+			(at 43.18 62.2299 90)
 			(show_name no)
 			(do_not_autoplace no)
@@
 		)
 		(property "Footprint" ""
-			(at 57.15 62.23 0)
+			(at 46.99 62.23 0)
 			(hide yes)
 			(show_name no)
@@
 		)
 		(property "Datasheet" ""
-			(at 57.15 62.23 0)
+			(at 46.99 62.23 0)
 			(hide yes)
 			(show_name no)
@@
 		)
 		(property "Description" "Power symbol creates a global label with name \"GND\" , ground"
-			(at 57.15 62.23 0)
+			(at 46.99 62.23 0)
 			(hide yes)
 			(show_name no)
@@
 	)
 	(symbol
+		(lib_id "power:PWR_FLAG")
+		(at 53.34 62.23 180)
+		(unit 1)
+		(body_style 1)
+		(exclude_from_sim no)
+		(in_bom yes)
+		(on_board yes)
+		(in_pos_files yes)
+		(dnp no)
+		(fields_autoplaced yes)
+		(property "Reference" "#FLG02"
+			(at 53.34 64.135 0)
+			(hide yes)
+			(show_name no)
+			(do_not_autoplace no)
+			(effects
+				(font
+					(size 1.27 1.27)
+				)
+			)
+		)
+		(property "Value" "PWR_FLAG"
+			(at 53.34 67.31 0)
+			(show_name no)
+			(do_not_autoplace no)
+			(effects
+				(font
+					(size 1.27 1.27)
+				)
+			)
+		)
+		(property "Footprint" ""
+			(at 53.34 62.23 0)
+			(hide yes)
+			(show_name no)
+			(do_not_autoplace no)
+			(effects
+				(font
+					(size 1.27 1.27)
+				)
+			)
+		)
+		(property "Datasheet" ""
+			(at 53.34 62.23 0)
+			(hide yes)
+			(show_name no)
+			(do_not_autoplace no)
+			(effects
+				(font
+					(size 1.27 1.27)
+				)
+			)
+		)
+		(property "Description" "Special symbol for telling ERC where power comes from"
+			(at 53.34 62.23 0)
+			(hide yes)
+			(show_name no)
+			(do_not_autoplace no)
+			(effects
+				(font
+					(size 1.27 1.27)
+				)
+			)
+		)
+		(pin "1"
+		)
+		(instances
+			(project "hacker-card"
+				(path "/8d7479d8-4d18-481b-a593-ed64f90da8e1"
+					(reference "#FLG02")
+					(unit 1)
+				)
+			)
+		)
+	)
+	(symbol
 		(lib_id "Device:R")
 		(at 82.55 86.36 0)
@@
 			)
 		)
-		(property "Value" "470"
+		(property "Value" "150"
 			(at 85.09 87.6299 0)
 			(show_name no)
@@
 			)
 		)
-		(property "LSC" "C23182"
+		(property "LSC" "C22808"
 			(at 82.55 86.36 0)
 			(hide yes)
@@
 			)
 		)
-		(property "Value" "470"
+		(property "Value" "150"
 			(at 71.12 87.6299 0)
 			(show_name no)
@@
 			)
 		)
-		(property "LSC" "C23182"
+		(property "LSC" "C22808"
 			(at 68.58 86.36 0)
 			(hide yes)
@@
 			)
 		)
-		(property "Value" "470"
+		(property "Value" "150"
 			(at 57.15 87.6299 0)
 			(show_name no)
@@
 			)
 		)
-		(property "LSC" "C23182"
+		(property "LSC" "C22808"
 			(at 54.61 86.36 0)
 			(hide yes)
@@
 					(unit 1)
 				)
+			)
+		)
+	)
+	(symbol
+		(lib_id "power:PWR_FLAG")
+		(at 83.82 62.23 180)
+		(unit 1)
+		(body_style 1)
+		(exclude_from_sim no)
+		(in_bom yes)
+		(on_board yes)
+		(in_pos_files yes)
+		(dnp no)
+		(property "Reference" "#FLG01"
+			(at 83.82 64.135 0)
+			(hide yes)
+			(show_name no)
+			(do_not_autoplace no)
+			(effects
+				(font
+					(size 1.27 1.27)
+				)
+			)
+		)
+		(property "Value" "PWR_FLAG"
+			(at 86.106 67.056 0)
+			(show_name no)
+			(do_not_autoplace no)
+			(effects
+				(font
+					(size 1.27 1.27)
+				)
+			)
+		)
+		(property "Footprint" ""
+			(at 83.82 62.23 0)
+			(hide yes)
+			(show_name no)
+			(do_not_autoplace no)
+			(effects
+				(font
+					(size 1.27 1.27)
+				)
+			)
+		)
+		(property "Datasheet" ""
+			(at 83.82 62.23 0)
+			(hide yes)
+			(show_name no)
+			(do_not_autoplace no)
+			(effects
+				(font
+					(size 1.27 1.27)
+				)
+			)
+		)
+		(property "Description" "Special symbol for telling ERC where power comes from"
+			(at 83.82 62.23 0)
+			(hide yes)
+			(show_name no)
+			(do_not_autoplace no)
+			(effects
+				(font
+					(size 1.27 1.27)
+				)
+			)
+		)
+		(pin "1"
+		)
+		(instances
+			(project "hacker-card"
+				(path "/8d7479d8-4d18-481b-a593-ed64f90da8e1"
+					(reference "#FLG01")
+					(unit 1)
+				)
